Commit message: Update package configuration for ROS2 Humble and Ignition Fortress: - Update CMakeLists.txt and package.xml - Add diff_drive_controller configuration - Add EKF configuration - Add world files - Update URDF with new colors and comments - Update launch file with bridge and controller configuration

File: urdf/assem_urdf.urdf.xacro (robot description, xacro)
@@ -1,4 +1,8 @@
 <?xml version="1.0" encoding="utf-8"?>
 <robot name="assem_urdf" xmlns:xacro="https://www.ros.org/wiki/xacro">
+  <!-- ============================================= -->
+  <!-- Base Component -->
+  <!-- ============================================= -->
+  <!-- Base link - Main body of the robot -->
   <link
     name="base_link">
@@ -26,7 +30,7 @@
       </geometry>
       <material
-        name="">
-        <color
-          rgba="1 1 1 1" />
+        name="base_material">
+        <color
+          rgba="0.2 0.2 0.2 1" /> <!-- Dark gray for base -->
       </material>
     </visual>
@@ -41,4 +45,8 @@
     </collision>
   </link>
+  <!-- ============================================= -->
+  <!-- Wheel Components -->
+  <!-- ============================================= -->
+  <!-- Right behind wheel -->
   <link
     name="right_behind_wheel">
@@ -66,7 +74,7 @@
       </geometry>
       <material
-        name="">
-        <color
-          rgba="0.79216 0.81961 0.93333 1" />
+        name="wheel_material">
+        <color
+          rgba="0.1 0.1 0.1 1" /> <!-- Black for wheels -->
       </material>
     </visual>
@@ -81,4 +89,5 @@
     </collision>
   </link>
+  <!-- Joint connecting right behind wheel to base -->
   <joint
     name="right_behind_wheel_joint"
@@ -94,4 +103,5 @@
       xyz="0 0 1" />
   </joint>
+  <!-- Left behind wheel -->
   <link
     name="left_behind_wheel">
@@ -119,7 +129,7 @@
       </geometry>
       <material
-        name="">
-        <color
-          rgba="0.79216 0.81961 0.93333 1" />
+        name="wheel_material">
+        <color
+          rgba="0.1 0.1 0.1 1" /> <!-- Black for wheels -->
       </material>
     </visual>
@@ -134,4 +144,5 @@
     </collision>
   </link>
+  <!-- Joint connecting left behind wheel to base -->
   <joint
     name="left_behind_wheel_joint"
@@ -147,4 +158,5 @@
       xyz="0 0 1" />
   </joint>
+  <!-- Right front wheel -->
   <link
     name="right_front_wheel">
@@ -172,7 +184,7 @@
       </geometry>
       <material
-        name="">
-        <color
-          rgba="0.79216 0.81961 0.93333 1" />
+        name="wheel_material">
+        <color
+          rgba="0.1 0.1 0.1 1" /> <!-- Black for wheels -->
       </material>
     </visual>
@@ -187,4 +199,5 @@
     </collision>
   </link>
+  <!-- Joint connecting right front wheel to base -->
   <joint
     name="right_front_wheel_joint"
@@ -200,4 +213,5 @@
       xyz="0 0 1" />
   </joint>
+  <!-- Left front wheel -->
   <link
     name="left_front_wheel">
@@ -225,7 +239,7 @@
       </geometry>
       <material
-        name="">
-        <color
-          rgba="0.79216 0.81961 0.93333 1" />
+        name="wheel_material">
+        <color
+          rgba="0.1 0.1 0.1 1" /> <!-- Black for wheels -->
       </material>
     </visual>
@@ -240,4 +254,5 @@
     </collision>
   </link>
+  <!-- Joint connecting left front wheel to base -->
   <joint
     name="left_front_wheel_joint"
@@ -253,4 +268,50 @@
       xyz="0 0 1" />
   </joint>
+  <ros2_control name="IgnitionSystem" type="system">
+    <hardware>
+      <plugin>ign_ros2_control/IgnitionSystem</plugin>
+    </hardware>
+    <joint name="left_front_wheel_joint">
+      <command_interface name="velocity">
+        <param name="min">-10</param>
+        <param name="max">10</param>
+      </command_interface>
+      <state_interface name="position"/>
+      <state_interface name="velocity"/>
+    </joint>
+    <joint name="right_front_wheel_joint">
+      <command_interface name="velocity">
+        <param name="min">-10</param>
+        <param name="max">10</param>
+      </command_interface>
+      <state_interface name="position"/>
+      <state_interface name="velocity"/>
+    </joint>
+    <joint name="left_rear_wheel_joint">
+      <command_interface name="velocity">
+        <param name="min">-10</param>
+        <param name="max">10</param>
+      </command_interface>
+      <state_interface name="position"/>
+      <state_interface name="velocity"/>
+    </joint>
+    <joint name="right_rear_wheel_joint">
+      <command_interface name="velocity">
+        <param name="min">-10</param>
+        <param name="max">10</param>
+      </command_interface>
+      <state_interface name="position"/>
+      <state_interface name="velocity"/>
+    </joint>
+  </ros2_control>
+  <gazebo>
+    <plugin filename="ign_ros2_control-system" name="ign_ros2_control::IgnitionROS2ControlPlugin">
+      <parameters>$(find assem_urdf)/config/diff_drive_controller_velocity.yaml</parameters>
+    </plugin>
+  </gazebo>
+  <!-- ============================================= -->
+  <!-- Sensor Components -->
+  <!-- ============================================= -->
+  <!-- Lidar sensor -->
   <link
     name="lidar">
@@ -278,7 +339,7 @@
       </geometry>
       <material
-        name="">
-        <color
-          rgba="0.75294 0.75294 0.75294 1" />
+        name="lidar_material">
+        <color
+          rgba="0.8 0.2 0.2 1" /> <!-- Red for lidar -->
       </material>
     </visual>
@@ -293,4 +354,5 @@
     </collision>
   </link>
+  <!-- Joint connecting lidar to base -->
   <joint
     name="lidar_joint"
@@ -311,4 +373,8 @@
       velocity="0" />
   </joint>
+  <!-- ============================================= -->
+  <!-- Manipulator Components -->
+  <!-- ============================================= -->
+  <!-- Right hand -->
   <link
     name="right_hand">
@@ -336,7 +402,7 @@
       </geometry>
       <material
-        name="">
-        <color
-          rgba="0.79216 0.81961 0.93333 1" />
+        name="hand_material">
+        <color
+          rgba="0.2 0.6 0.8 1" /> <!-- Blue for hands -->
       </material>
     </visual>
@@ -351,4 +417,5 @@
     </collision>
   </link>
+  <!-- Joint connecting right hand to lidar -->
   <joint
     name="right_hand_joint"
@@ -369,4 +436,5 @@
       velocity="0" />
   </joint>
+  <!-- Left hand -->
   <link
     name="left_hand">
@@ -394,7 +462,7 @@
       </geometry>
       <material
-        name="">
-        <color
-          rgba="0.79216 0.81961 0.93333 1" />
+        name="hand_material">
+        <color
+          rgba="0.2 0.6 0.8 1" /> <!-- Blue for hands -->
       </material>
     </visual>
@@ -409,4 +477,5 @@
     </collision>
   </link>
+  <!-- Joint connecting left hand to lidar -->
   <joint
     name="left_hand_joint"
@@ -427,4 +496,8 @@
       velocity="0" />
   </joint>
+  <!-- ============================================= -->
+  <!-- Leg Components -->
+  <!-- ============================================= -->
+  <!-- Right leg -->
   <link
     name="right_leg">
@@ -452,7 +525,7 @@
       </geometry>
       <material
-        name="">
-        <color
-          rgba="0.79216 0.81961 0.93333 1" />
+        name="leg_material">
+        <color
+          rgba="0.4 0.4 0.4 1" /> <!-- Medium gray for legs -->
       </material>
     </visual>
@@ -467,4 +540,5 @@
     </collision>
   </link>
+  <!-- Joint connecting right leg to lidar -->
   <joint
     name="right_leg_joint"
@@ -485,4 +559,5 @@
       velocity="0" />
   </joint>
+  <!-- Left leg -->
   <link
     name="left_leg">
@@ -510,7 +585,7 @@
       </geometry>
       <material
-        name="">
-        <color
-          rgba="0.79216 0.81961 0.93333 1" />
+        name="leg_material">
+        <color
+          rgba="0.4 0.4 0.4 1" /> <!-- Medium gray for legs -->
       </material>
     </visual>
@@ -525,4 +600,5 @@
     </collision>
   </link>
+  <!-- Joint connecting left leg to lidar -->
   <joint
     name="left_leg_joint"
@@ -543,4 +619,8 @@
       velocity="0" />
   </joint>
+  <!-- ============================================= -->
+  <!-- Head Component -->
+  <!-- ============================================= -->
+  <!-- Head -->
   <link
     name="head_link">
@@ -568,7 +648,7 @@
       </geometry>
       <material
-        name="">
-        <color
-          rgba="0.79216 0.81961 0.93333 1" />
+        name="head_material">
+        <color
+          rgba="0.8 0.8 0.2 1" /> <!-- Yellow for head -->
       </material>
     </visual>
@@ -583,4 +663,5 @@
     </collision>
   </link>
+  <!-- Joint connecting head to lidar -->
   <joint
     name="head_joint"

Commit message: fig_bug

File: urdf/assem_urdf.urdf.xacro (robot description, xacro)
@@ -45,4 +45,16 @@
     </collision>
   </link>
+  <!-- Robot Footprint -->
+  <link name="base_footprint">
+    <inertial>
+      <mass value="0.0001"/>
+      <inertia ixx="0.0001" ixy="0.0" ixz="0.0" iyy="0.0001" iyz="0.0" izz="0.0001"/>
+    </inertial>
+  </link>
+  <joint name="base_joint" type="fixed">
+    <parent link="base_footprint"/>
+    <child link="base_link"/>
+    <origin xyz="0.0 0.0 0.1" rpy="0 0 0"/>
+  </joint>
   <!-- ============================================= -->
   <!-- Wheel Components -->

Commit message: Update robot configuration and remove unused files

File: urdf/assem_urdf.urdf.xacro (robot description, xacro)
@@ -2,22 +2,21 @@
 <robot name="assem_urdf" xmlns:xacro="https://www.ros.org/wiki/xacro">
   <!-- ============================================= -->
-  <!-- Base Component -->
-  <!-- ============================================= -->
-  <!-- Base link - Main body of the robot -->
+  <!-- Base Link - Main body of the robot           -->
+  <!-- ============================================= -->
   <link
     name="base_link">
     <inertial>
       <origin
-        xyz="0.00023393 5.2019E-06 0.045075"
+        xyz="0.0099132 0.00030561 0.03955"
         rpy="0 0 0" />
       <mass
         value="5" />
       <inertia
-        ixx="0.036016"
-        ixy="7.4282E-07"
-        ixz="2.6297E-05"
-        iyy="0.034799"
-        iyz="-1.3398E-07"
-        izz="0.068467" />
+        ixx="0.0013702"
+        ixy="9.6491E-08"
+        ixz="1.1654E-07"
+        iyy="0.0013447"
+        iyz="3.7844E-07"
+        izz="0.0026486" />
     </inertial>
     <visual>
@@ -30,7 +29,7 @@
       </geometry>
       <material
-        name="base_material">
-        <color
-          rgba="0.2 0.2 0.2 1" /> <!-- Dark gray for base -->
+        name="">
+        <color
+          rgba="0.2 0.2 0.8 1" />
       </material>
     </visual>
@@ -45,34 +44,21 @@
     </collision>
   </link>
-  <!-- Robot Footprint -->
-  <link name="base_footprint">
-    <inertial>
-      <mass value="0.0001"/>
-      <inertia ixx="0.0001" ixy="0.0" ixz="0.0" iyy="0.0001" iyz="0.0" izz="0.0001"/>
-    </inertial>
-  </link>
-  <joint name="base_joint" type="fixed">
-    <parent link="base_footprint"/>
-    <child link="base_link"/>
-    <origin xyz="0.0 0.0 0.1" rpy="0 0 0"/>
-  </joint>
-  <!-- ============================================= -->
-  <!-- Wheel Components -->
-  <!-- ============================================= -->
-  <!-- Right behind wheel -->
-  <link
-    name="right_behind_wheel">
-    <inertial>
-      <origin
-        xyz="0 0 -1.3878E-17"
-        rpy="0 0 0" />
-      <mass
-        value="3" />
+  <!-- ============================================= -->
+  <!-- Right Wheel - Drive mechanism                -->
+  <!-- ============================================= -->
+  <link
+    name="wheel_right_link">
+    <inertial>
+      <origin
+        xyz="-6.9389E-18 -3.4694E-18 -1.3878E-17"
+        rpy="0 0 0" />
+      <mass
+        value="0.1" />
       <inertia
         ixx="2.8744E-05"
-        ixy="-2.5643E-21"
-        ixz="-4.7646E-23"
+        ixy="-7.5972E-22"
+        ixz="2.3823E-23"
         iyy="2.8744E-05"
-        iyz="-1.3124E-37"
+        iyz="-2.9779E-24"
         izz="4.7183E-05" />
     </inertial>
@@ -83,233 +69,107 @@
       <geometry>
         <mesh
-          filename="file://$(find assem_urdf)/meshes/right_behind_wheel.STL" />
-      </geometry>
-      <material
-        name="wheel_material">
-        <color
-          rgba="0.1 0.1 0.1 1" /> <!-- Black for wheels -->
-      </material>
-    </visual>
-    <collision>
-      <origin
-        xyz="0 0 0"
-        rpy="0 0 0" />
-      <geometry>
-        <mesh
-          filename="file://$(find assem_urdf)/meshes/right_behind_wheel.STL" />
-      </geometry>
-    </collision>
-  </link>
-  <!-- Joint connecting right behind wheel to base -->
+          filename="file://$(find assem_urdf)/meshes/wheel_right_link.STL" />
+      </geometry>
+      <material
+        name="">
+        <color
+          rgba="0.8 0.2 0.2 1" />
+      </material>
+    </visual>
+    <collision>
+      <origin
+        xyz="0 0 0"
+        rpy="0 0 0" />
+      <geometry>
+        <mesh
+          filename="file://$(find assem_urdf)/meshes/wheel_right_link.STL" />
+      </geometry>
+    </collision>
+  </link>
   <joint
-    name="right_behind_wheel_joint"
+    name="wheel_right_joint"
     type="continuous">
     <origin
-      xyz="-0.11 -0.099999 0.0198"
+      xyz="-0.036511 -0.099997 0.0198"
+      rpy="1.5708 0 0" />
+    <parent
+      link="base_link" />
+    <child
+      link="wheel_right_link" />
+    <axis
+      xyz="0 0 -1" />
+  </joint>
+  <!-- ============================================= -->
+  <!-- Left Wheel - Drive mechanism                 -->
+  <!-- ============================================= -->
+  <link
+    name="wheel_left_link">
+    <inertial>
+      <origin
+        xyz="-6.9389E-18 -3.4694E-18 1.3878E-17"
+        rpy="0 0 0" />
+      <mass
+        value="0.1" />
+      <inertia
+        ixx="2.8744E-05"
+        ixy="-7.5972E-22"
+        ixz="-2.3823E-23"
+        iyy="2.8744E-05"
+        iyz="2.9779E-24"
+        izz="4.7183E-05" />
+    </inertial>
+    <visual>
+      <origin
+        xyz="0 0 0"
+        rpy="0 0 0" />
+      <geometry>
+        <mesh
+          filename="file://$(find assem_urdf)/meshes/wheel_left_link.STL" />
+      </geometry>
+      <material
+        name="">
+        <color
+          rgba="0.8 0.2 0.2 1" />
+      </material>
+    </visual>
+    <collision>
+      <origin
+        xyz="0 0 0"
+        rpy="0 0 0" />
+      <geometry>
+        <mesh
+          filename="file://$(find assem_urdf)/meshes/wheel_left_link.STL" />
+      </geometry>
+    </collision>
+  </link>
+  <joint
+    name="wheel_left_joint"
+    type="continuous">
+    <origin
+      xyz="-0.036511 0.099997 0.0198"
       rpy="-1.5708 0 0" />
     <parent
       link="base_link" />
     <child
-      link="right_behind_wheel" />
+      link="wheel_left_link" />
     <axis
       xyz="0 0 1" />
   </joint>
-  <!-- Left behind wheel -->
-  <link
-    name="left_behind_wheel">
-    <inertial>
-      <origin
-        xyz="0 0 0"
-        rpy="0 0 0" />
-      <mass
-        value="3" />
-      <inertia
-        ixx="2.8744E-05"
-        ixy="-3.2552E-21"
-        ixz="4.7646E-23"
-        iyy="2.8744E-05"
-        iyz="-1.1911E-23"
-        izz="4.7183E-05" />
-    </inertial>
-    <visual>
-      <origin
-        xyz="0 0 0"
-        rpy="0 0 0" />
-      <geometry>
-        <mesh
-          filename="file://$(find assem_urdf)/meshes/left_behind_wheel.STL" />
-      </geometry>
-      <material
-        name="wheel_material">
-        <color
-          rgba="0.1 0.1 0.1 1" /> <!-- Black for wheels -->
-      </material>
-    </visual>
-    <collision>
-      <origin
-        xyz="0 0 0"
-        rpy="0 0 0" />
-      <geometry>
-        <mesh
-          filename="file://$(find assem_urdf)/meshes/left_behind_wheel.STL" />
-      </geometry>
-    </collision>
-  </link>
-  <!-- Joint connecting left behind wheel to base -->
-  <joint
-    name="left_behind_wheel_joint"
-    type="continuous">
-    <origin
-      xyz="-0.110001193758665 0.100001193758665 0.0198"
-      rpy="-1.5707963267949 0 0" />
-    <parent
-      link="base_link" />
-    <child
-      link="left_behind_wheel" />
-    <axis
-      xyz="0 0 1" />
-  </joint>
-  <!-- Right front wheel -->
-  <link
-    name="right_front_wheel">
-    <inertial>
-      <origin
-        xyz="0 0 -1.3878E-17"
-        rpy="0 0 0" />
-      <mass
-        value="3" />
-      <inertia
-        ixx="2.8744E-05"
-        ixy="3.2552E-21"
-        ixz="4.7646E-23"
-        iyy="2.8744E-05"
-        iyz="1.1911E-23"
-        izz="4.7183E-05" />
-    </inertial>
-    <visual>
-      <origin
-        xyz="0 0 0"
-        rpy="0 0 0" />
-      <geometry>
-        <mesh
-          filename="file://$(find assem_urdf)/meshes/right_front_wheel.STL" />
-      </geometry>
-      <material
-        name="wheel_material">
-        <color
-          rgba="0.1 0.1 0.1 1" /> <!-- Black for wheels -->
-      </material>
-    </visual>
-    <collision>
-      <origin
-        xyz="0 0 0"
-        rpy="0 0 0" />
-      <geometry>
-        <mesh
-          filename="file://$(find assem_urdf)/meshes/right_front_wheel.STL" />
-      </geometry>
-    </collision>
-  </link>
-  <!-- Joint connecting right front wheel to base -->
-  <joint
-    name="right_front_wheel_joint"
-    type="continuous">
-    <origin
-      xyz="0.109998806241335 -0.0999988062413351 0.0198"
-      rpy="-1.5707963267949 0 0" />
-    <parent
-      link="base_link" />
-    <child
-      link="right_front_wheel" />
-    <axis
-      xyz="0 0 1" />
-  </joint>
-  <!-- Left front wheel -->
-  <link
-    name="left_front_wheel">
-    <inertial>
-      <origin
-        xyz="0 0 0"
-        rpy="0 0 0" />
-      <mass
-        value="3" />
-      <inertia
-        ixx="2.8744E-05"
-        ixy="2.5643E-21"
-        ixz="-4.7646E-23"
-        iyy="2.8744E-05"
-        iyz="1.3124E-37"
-        izz="4.7183E-05" />
-    </inertial>
-    <visual>
-      <origin
-        xyz="0 0 0"
-        rpy="0 0 0" />
-      <geometry>
-        <mesh
-          filename="file://$(find assem_urdf)/meshes/left_front_wheel.STL" />
-      </geometry>
-      <material
-        name="wheel_material">
-        <color
-          rgba="0.1 0.1 0.1 1" /> <!-- Black for wheels -->
-      </material>
-    </visual>
-    <collision>
-      <origin
-        xyz="0 0 0"
-        rpy="0 0 0" />
-      <geometry>
-        <mesh
-          filename="file://$(find assem_urdf)/meshes/left_front_wheel.STL" />
-      </geometry>
-    </collision>
-  </link>
-  <!-- Joint connecting left front wheel to base -->
-  <joint
-    name="left_front_wheel_joint"
-    type="continuous">
-    <origin
-      xyz="0.109998806241335 0.100001193758665 0.0198"
-      rpy="-1.5707963267949 0 0" />
-    <parent
-      link="base_link" />
-    <child
-      link="left_front_wheel" />
-    <axis
-      xyz="0 0 1" />
-  </joint>
-  <ros2_control name="IgnitionSystem" type="system">
+  <!-- <ros2_control name="IgnitionSystem" type="system">
     <hardware>
       <plugin>ign_ros2_control/IgnitionSystem</plugin>
     </hardware>
-    <joint name="left_front_wheel_joint">
+    <joint name="wheel_left_joint">
       <command_interface name="velocity">
-        <param name="min">-10</param>
-        <param name="max">10</param>
+        <param name="min">-1</param>
+        <param name="max">1</param>
       </command_interface>
       <state_interface name="position"/>
       <state_interface name="velocity"/>
     </joint>
-    <joint name="right_front_wheel_joint">
+    <joint name="wheel_right_joint">
       <command_interface name="velocity">
-        <param name="min">-10</param>
-        <param name="max">10</param>
-      </command_interface>
-      <state_interface name="position"/>
-      <state_interface name="velocity"/>
-    </joint>
-    <joint name="left_rear_wheel_joint">
-      <command_interface name="velocity">
-        <param name="min">-10</param>
-        <param name="max">10</param>
-      </command_interface>
-      <state_interface name="position"/>
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